Commit message: switch to galactic

File: src/maze_bringup/urdf/rosbot.urdf (robot description, URDF)
Before this commit: robot rosbot, 15 links, 14 joints
Links:
- link base_link: geometry collision box size=0.20 0.15 0.04; visual mesh filename=package://maze_bringup/meshes/box.dae scale=0.001 0.001 0.001
- link camera_link: geometry collision box size=0.001 0.001 0.001; visual mesh filename=package://maze_bringup/meshes/astra.dae scale=0.001 0.001 0.001
- link front_left_wheel: geometry collision mesh filename=package://maze_bringup/meshes/wheel-v2.stl scale=0.001 0.001 0.001; visual mesh filename=package://maze_bringup/meshes/wheel.dae scale=0.001 0.001 0.001
- link front_right_wheel: geometry collision mesh filename=package://maze_bringup/meshes/wheel-v2.stl scale=0.001 0.001 0.001; visual mesh filename=package://maze_bringup/meshes/wheel.dae scale=0.001 0.001 0.001
- link laser: geometry collision mesh filename=package://maze_bringup/meshes/rplidar.dae scale=0.001 0.001 0.001; visual mesh filename=package://maze_bringup/meshes/rplidar.dae scale=0.001 0.001 0.001
- link rear_left_wheel: geometry collision mesh filename=package://maze_bringup/meshes/wheel-v2.stl scale=0.001 0.001 0.001; visual mesh filename=package://maze_bringup/meshes/wheel.dae scale=0.001 0.001 0.001
- link rear_right_wheel: geometry collision mesh filename=package://maze_bringup/meshes/wheel-v2.stl scale=0.001 0.001 0.001; visual mesh filename=package://maze_bringup/meshes/wheel.dae scale=0.001 0.001 0.001
- link top: geometry visual mesh filename=package://maze_bringup/meshes/upper.dae scale=0.001 0.001 0.001
