Commit message: rosbot xacro file for simulation

File: src/maze_bringup/urdf/rosbot.xacro (robot description, xacro)
@@ -6,7 +6,7 @@
   <xacro:property name="cameraMass" value="0.1"/>
   <xacro:property name="namespace" value="$(arg robot_namespace)" />
-  <xacro:include filename="$(find rosbot_description)/urdf/rosbot.gazebo" />
-  <xacro:include filename="$(find rosbot_description)/urdf/materials.xacro" />
-  <xacro:include filename="$(find rosbot_description)/urdf/macros.xacro" />
+  <xacro:include filename="$(find maze_bringup)/urdf/rosbot.gazebo" />
+  <xacro:include filename="$(find maze_bringup)/urdf/materials.xacro" />
+  <xacro:include filename="$(find maze_bringup)/urdf/macros.xacro" />
   <link name="dummy"></link>
   <joint name="dummy_joint" type="fixed">
@@ -34,5 +34,5 @@
       <origin xyz="0 0 -0.02" rpy=" 1.5707 0 1.5707"/>
       <geometry>
-        <mesh filename="package://rosbot_description/meshes/box.dae" scale="0.001 0.001 0.001" />
+        <mesh filename="package://maze_bringup/meshes/box.dae" scale="0.001 0.001 0.001" />
       </geometry>
     </visual>
@@ -58,5 +58,5 @@
       <origin xyz="0 0 0.055" rpy=" 1.5707 0 1.5707"/>
       <geometry>
-        <mesh filename="package://rosbot_description/meshes/upper.dae" scale="0.001 0.001 0.001" />
+        <mesh filename="package://maze_bringup/meshes/upper.dae" scale="0.001 0.001 0.001" />
       </geometry>
     </visual>
@@ -66,5 +66,5 @@
       <origin xyz="0 0 0" rpy="0 0 1.5707"/>
       <geometry>
-        <mesh filename="package://rosbot_description/meshes/wheel-v2.stl" scale="0.001 0.001 0.001" />
+        <mesh filename="package://maze_bringup/meshes/wheel-v2.stl" scale="0.001 0.001 0.001" />
       </geometry>
       <surface>
@@ -80,5 +80,5 @@
       <origin xyz="0 0 0" rpy="0 0 1.5707"/>
       <geometry>
-        <mesh filename="package://rosbot_description/meshes/wheel.dae" scale="0.001 0.001 0.001" />
+        <mesh filename="package://maze_bringup/meshes/wheel.dae" scale="0.001 0.001 0.001" />
       </geometry>
     </visual>
@@ -96,5 +96,5 @@
       <origin xyz="0 0 0" rpy="0 0 -1.5707"/>
       <geometry>
-        <mesh filename="package://rosbot_description/meshes/wheel-v2.stl" scale="0.001 0.001 0.001" />
+        <mesh filename="package://maze_bringup/meshes/wheel-v2.stl" scale="0.001 0.001 0.001" />
       </geometry>
       <surface>
@@ -110,5 +110,5 @@
       <origin xyz="0 0 0" rpy="0 0 -1.5707"/>
       <geometry>
-        <mesh filename="package://rosbot_description/meshes/wheel.dae" scale="0.001 0.001 0.001" />
+        <mesh filename="package://maze_bringup/meshes/wheel.dae" scale="0.001 0.001 0.001" />
       </geometry>
     </visual>
@@ -126,5 +126,5 @@
       <origin xyz="0 0 0" rpy="0 0 1.5707"/>
       <geometry>
-        <mesh filename="package://rosbot_description/meshes/wheel-v2.stl" scale="0.001 0.001 0.001" />
+        <mesh filename="package://maze_bringup/meshes/wheel-v2.stl" scale="0.001 0.001 0.001" />
       </geometry>
       <surface>
@@ -140,5 +140,5 @@
       <origin xyz="0 0 0" rpy="0 0 1.5707"/>
       <geometry>
-        <mesh filename="package://rosbot_description/meshes/wheel.dae" scale="0.001 0.001 0.001" />
+        <mesh filename="package://maze_bringup/meshes/wheel.dae" scale="0.001 0.001 0.001" />
       </geometry>
     </visual>
@@ -156,5 +156,5 @@
       <origin xyz="0 0 0" rpy="0 0 -1.5707"/>
       <geometry>
-        <mesh filename="package://rosbot_description/meshes/wheel-v2.stl" scale="0.001 0.001 0.001" />
+        <mesh filename="package://maze_bringup/meshes/wheel-v2.stl" scale="0.001 0.001 0.001" />
       </geometry>
       <surface>
@@ -170,5 +170,5 @@
       <origin xyz="0 0 0" rpy="0 0 -1.5707"/>
       <geometry>
-        <mesh filename="package://rosbot_description/meshes/wheel.dae" scale="0.001 0.001 0.001" />
+        <mesh filename="package://maze_bringup/meshes/wheel.dae" scale="0.001 0.001 0.001" />
       </geometry>
     </visual>
@@ -267,5 +267,5 @@
       <origin xyz="-0.01 0 -0.03" rpy="1.5707 0 1.5707"/>
       <geometry>
-        <mesh filename="package://rosbot_description/meshes/astra.dae" scale="0.001 0.001 0.001" />
+        <mesh filename="package://maze_bringup/meshes/astra.dae" scale="0.001 0.001 0.001" />
       </geometry>
     </visual>
@@ -301,5 +301,5 @@
       <origin xyz="0 0 0" rpy="1.5707 0 4.71"/>
       <geometry>
-        <mesh filename="package://rosbot_description/meshes/rplidar.dae" scale="0.001 0.001 0.001" />
+        <mesh filename="package://maze_bringup/meshes/rplidar.dae" scale="0.001 0.001 0.001" />
       </geometry>
     </collision>
@@ -307,5 +307,5 @@
       <origin xyz="0 0 0" rpy="1.5707 0 4.71"/>
       <geometry>
-        <mesh filename="package://rosbot_description/meshes/rplidar.dae" scale="0.001 0.001 0.001" />
+        <mesh filename="package://maze_bringup/meshes/rplidar.dae" scale="0.001 0.001 0.001" />
       </geometry>
     </visual>
